File: Skizzen/Schaltplan/Schaltplan.kicad_pcb (KiCad board)
At the start: 2 copper layers, 52 parts, among them J1 I2C Sensor, J10 max. 250VAC/5A, J2 I2C Sensor, J3 I2C Sensor, J4 I2C Sensor, J5 I2C Sensor, J6 I2C Sensor, J7 12V DC, 2A, J8 max. 30VDC/2A, J9 max. 250VAC/5A, K1 G5LE-1, K2 G5LE-1, K3 G6S-2, M1 FAN0, M2 FAN1, M3 FAN2, Q1 2N7000, Q10 IRF9540N, Q11 IRF9540N, Q12 IRF9540N, Q13 2N7000, Q14 2N7000, Q15 2N7000, Q2 2N7000, Q3 2N7000, Q4 2N7000, Q5 2N7000, Q6 2N7000, Q7 2N7000, Q8 2N7000, Q9 2N7000, SW1 CFG_MODE, U1 NodeMCU_1.0_(ESP-12E), U2 TCA9548A, U3 RIT276-OLED-Display, U4 LM7805_TO220

Commit message: Woche 9 17.10.2021 - 24.10.2021
Parts:
- J7: footprint Jumper:SolderJumper-3_P1.3mm_Bridged12_Pad1.0x1.5mm -> KL:Buchse
- moved SW1 147.0 mm to (82.5, 73.7)
- moved J9 135.5 mm to (246.4, 111.8), turned to 90 degrees
- moved K3 124.2 mm to (204.5, 129.5)
- moved Q9 117.4 mm to (139.7, 53.3), turned to 90 degrees
- moved Q4 111.0 mm to (134.6, 69.8), turned to 90 degrees
- moved Q3 103.8 mm to (142.2, 66.0), turned to 90 degrees
- moved R2 102.9 mm to (128.3, 82.5)
- moved Q2 101.6 mm to (134.6, 88.9), turned to 90 degrees
- moved Q7 101.1 mm to (141.0, 91.4), turned to 90 degrees
- moved R3 100.0 mm to (135.9, 63.5), turned to 180 degrees
- moved Q8 97.7 mm to (142.2, 72.4), turned to 90 degrees
- moved U3 94.9 mm to (157.5, 104.1)
- moved R11 94.3 mm to (190.5, 133.3), turned to 180 degrees
- moved Q1 92.2 mm to (141.0, 85.1), turned to 90 degrees
- moved R4 91.2 mm to (133.3, 44.5), turned to 180 degrees
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Connections:
- C2 pad 1: Net-(C2-Pad1) -> Net-(C1-Pad1)
- Q11 pad 2: Net-(C2-Pad1) -> Net-(C1-Pad1)
- R7 pad 1: Net-(C2-Pad1) -> Net-(C1-Pad1)
Routing:
- net GND: track 187.8 -> 965.3 mm
- net Net-(C1-Pad1): track 0.00 -> 448.9 mm
- net Net-(Q15-Pad2): track 0.00 -> 184.1 mm
- net Net-(C4-Pad1): track 0.00 -> 115.7 mm
- net Net-(Q6-Pad2): track 0.00 -> 107.5 mm
- net Net-(Q13-Pad2): track 0.00 -> 89.9 mm
- net Net-(Q4-Pad2): track 0.00 -> 78.7 mm
- net Net-(R1-Pad2): track 0.00 -> 70.0 mm
- net Net-(J9-Pad1): track 0.00 -> 67.9 mm
- net Net-(M1-Pad4): track 0.00 -> 59.3 mm
- net Net-(Q2-Pad2): track 0.00 -> 55.6 mm
- net Net-(M2-Pad4): track 0.00 -> 55.1 mm
- net Net-(M3-Pad4): track 0.00 -> 49.8 mm
- net Net-(J10-Pad2): track 0.00 -> 45.3 mm
- net Net-(J8-Pad1): track 0.00 -> 43.6 mm
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
Commit message: Woche 20 02.01.2022 - 08.01.2022
Parts:
- removed J2, J3, J4, J5, J6: I2C Sensor, Sensor:Aosong_DHT11_5.5x12.0_P2.54mm
- added H1: MountingHole, MountingHole:MountingHole_3.2mm_M3, F.Cu at (78.7, 139.7)
- added H2: MountingHole, MountingHole:MountingHole_3.2mm_M3, F.Cu at (228.6, 139.7)
- added H3: MountingHole, MountingHole:MountingHole_3.2mm_M3, F.Cu at (228.6, 48.3)
- added H4: MountingHole, MountingHole:MountingHole_3.2mm_M3, F.Cu at (78.7, 48.3)
- added U5: YAAJ_DCDC_StepDown_LM2596, LM2596Module:YAAJ_DCDC_StepDown_LM2596, F.Cu at (137.2, 138.4)
- C5: footprint Capacitor_THT:C_Disc_D3.0mm_W1.6mm_P2.50mm -> Capacitor_THT:CP_Radial_Tantal_D4.5mm_P5.00mm
- J1: value I2C Sensor -> Conn_02x24_Counter_Clockwise; footprint Sensor:Aosong_DHT11_5.5x12.0_P2.54mm -> Terminals:FFKDSH-2,54_24
- J7: footprint KL:Buchse -> Connector_PinHeader_2.54mm:PinHeader_1x03_P2.54mm_Vertical; moved to B.Cu
- M1: value FAN0 -> FAN1
- M2: value FAN1 -> FAN2
- M3: value FAN2 -> FAN3
- R1, R2, R4, R5, R7, R9: footprint Resistor_THT:R_Axial_DIN0204_L3.6mm_D1.6mm_P7.62mm_Horizontal -> Resistor_THT:R_Axial_DIN0204_L3.6mm_D1.6mm_P2.54mm_Vertical
- R11: footprint Resistor_THT:R_Axial_DIN0207_L6.3mm_D2.5mm_P7.62mm_Horizontal -> Resistor_THT:R_Axial_DIN0204_L3.6mm_D1.6mm_P2.54mm_Vertical
- R3: footprint Resistor_THT:R_Axial_DIN0204_L3.6mm_D1.6mm_P7.62mm_Horizontal -> Resistor_THT:R_Axial_DIN0204_L3.6mm_D1.6mm_P2.54mm_Vertical; moved to B.Cu
- U2: value TCA9548A -> TCA9548A_Breakout; footprint KL:TCA9548A -> KL:TCA9548A_Breakout
- U3: footprint Connector_PinHeader_2.54mm:PinHeader_1x04_P2.54mm_Vertical -> Oled-Display:SSD1306_128x64_0.96
- moved U4 118.6 mm to (111.8, 129.5), turned to 90 degrees
- moved C5 109.6 mm to (121.9, 129.5)
- moved C4 103.4 mm to (105.4, 120.7), turned to 180 degrees
- moved J7 100.0 mm to (146.1, 134.6), turned to 0 degrees
- moved M3 98.6 mm to (196.8, 138.4), turned to 270 degrees
- moved R4 94.7 mm to (200.0, 111.8), turned to 90 degrees
- moved R9 91.6 mm to (197.5, 120.7), turned to 180 degrees
- moved C3 89.5 mm to (198.8, 124.5), turned to 180 degrees
- moved Q12 86.8 mm to (191.8, 133.3), turned to 0 degrees
- moved Q6 86.4 mm to (201.9, 101.6), turned to 270 degrees
- moved Q5 83.5 mm to (192.4, 111.8)
- moved R10 82.1 mm to (188.6, 124.5), turned to 90 degrees
- moved M2 76.6 mm to (179.1, 138.4), turned to 270 degrees
- moved Q9 71.9 mm to (193.0, 101.6), turned to 270 degrees
- moved R3 66.5 mm to (181.0, 112.4), turned to 90 degrees
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Connections:
- net Net-(C4-Pad1) renamed /V5V0
- net Net-(Q1-Pad2) renamed /FAN1_PWM#
- net Net-(Q15-Pad2) renamed /ESP_CIRC_ON
- net Net-(Q2-Pad2) renamed /ESP_FAN1_PWM
- net Net-(Q3-Pad2) renamed /FAN2_PWM#
- net Net-(Q4-Pad2) renamed /ESP_FAN2_PWM
- net Net-(Q5-Pad2) renamed /FAN3_PWM#
- C1 pad 1: Net-(C1-Pad1) -> /V12V0IN
- C2 pad 1: Net-(C1-Pad1) -> /V12V0IN
- C3 pad 1: Net-(C1-Pad1) -> /V12V0IN
- C5 pad 1: Net-(C1-Pad1) -> /V12V0IN
- J1 pad 2: Net-(J1-Pad2) -> /V3V3
- J7 pad 1: Net-(C1-Pad1) -> /V12V0IN
- J8 pad 1: Net-(J8-Pad1) -> /TANK_FULL_CLOSE
- J8 pad 2: Net-(J8-Pad2) -> /TANK_FULL_COMMON
- K1 pad 2: Net-(K1-Pad2) -> /V12V0IN
- K1 pad 5: Net-(C1-Pad1) -> Net-(K1-Pad5)
- K2 pad 5: Net-(C1-Pad1) -> /V12V0IN
- K3 pad 1: Net-(C1-Pad1) -> /V12V0IN
- K3 pad 10: Net-(J8-Pad1) -> Net-(J8-Pad3)
- K3 pad 8: Net-(J8-Pad2) -> /TANK_FULL_CLOSE
- K3 pad 9: Net-(J8-Pad3) -> /TANK_FULL_COMMON
- M1 pad 2: Net-(M1-Pad2) -> /FAN1_V12V0
- M1 pad 4: Net-(M1-Pad4) -> /FAN1_PWM
- M2 pad 2: Net-(M2-Pad2) -> /FAN2_V12V0
- M2 pad 4: Net-(M2-Pad4) -> /FAN2_PWM
- M3 pad 4: Net-(M3-Pad4) -> /FAN3_PWM
- Q1 pad 3: Net-(M1-Pad4) -> /FAN1_PWM
- Q10 pad 2: Net-(C1-Pad1) -> /FAN1_V12V0
- Q10 pad 3: Net-(M1-Pad2) -> /V12V0IN
- Q11 pad 2: Net-(C1-Pad1) -> /FAN2_V12V0
- Q11 pad 3: Net-(M2-Pad2) -> /V12V0IN
- Q12 pad 2: Net-(C1-Pad1) -> Net-(M3-Pad2)
- Q12 pad 3: Net-(M3-Pad2) -> /V12V0IN
- Q13 pad 2: Net-(Q13-Pad2) -> /ESP_DEHUM_ON
- Q14 pad 2: Net-(Q13-Pad2) -> /ESP_DEHUM_ON
- Q14 pad 3: Net-(K1-Pad2) -> Net-(K1-Pad5)
- Q3 pad 3: Net-(M2-Pad4) -> /FAN2_PWM
- Q5 pad 3: Net-(M3-Pad4) -> /FAN3_PWM
- Q6 pad 2: Net-(Q6-Pad2) -> /ESP_FAN3_PWM
- Q9 pad 2: Net-(Q6-Pad2) -> /ESP_FAN3_PWM
- R1 pad 1: Net-(J1-Pad2) -> /V3V3
- R1 pad 2: Net-(R1-Pad2) -> /ESP_FORCE_CFG_MODE
- R2 pad 1: Net-(M1-Pad4) -> /V12V0IN
- R3 pad 1: Net-(M2-Pad4) -> /V12V0IN
- R4 pad 1: Net-(M3-Pad4) -> /V12V0IN
- R5 pad 1: Net-(C1-Pad1) -> /V12V0IN
- R7 pad 1: Net-(C1-Pad1) -> /V12V0IN
- R9 pad 1: Net-(C1-Pad1) -> /V12V0IN
- SW1 pad 1: Net-(R1-Pad2) -> /ESP_FORCE_CFG_MODE
- U1 pad 11: Net-(J1-Pad2) -> /V3V3
- U1 pad 16: Net-(J1-Pad2) -> /V3V3
- U1 pad 20: Net-(R1-Pad2) -> /ESP_FAN3_PWM
- U1 pad 21: Net-(Q6-Pad2) -> /ESP_FORCE_CFG_MODE
- U1 pad 25: Net-(J1-Pad2) -> /V3V3
- U1 pad 26: Net-(Q13-Pad2) -> Net-(U1-Pad26)
- U1 pad 28: Net-(U1-Pad28) -> /ESP_SDA
- U1 pad 29: Net-(U1-Pad29) -> /ESP_SCL
- U1 pad 4: Net-(U1-Pad4) -> /ESP_DEHUM_ON
- U2 pad 1: Net-(J1-Pad4) -> /V3V3
- U2 pad 13: Net-(J6-Pad3) -> /MUX_SDA2
- U2 pad 14: Net-(U2-Pad14) -> /MUX_SCL2
- U2 pad 15: Net-(U2-Pad15) -> /MUX_SDA3
- U2 pad 16: Net-(U2-Pad16) -> /MUX_SCL3
- U2 pad 17: Net-(U2-Pad17) -> /MUX_SDA4
- U2 pad 18: GND -> /MUX_SCL4
- U2 pad 19: Net-(U1-Pad29) -> /MUX_SDA5
- U2 pad 2: Net-(J1-Pad3) -> GND
- U2 pad 20: Net-(U1-Pad28) -> /MUX_SCL5
- U2 pad 21: Net-(J1-Pad2) -> /MUX_SDA6
- U2 pad 22: Net-(J1-Pad2) -> /MUX_SCL6
- U2 pad 23: GND -> /MUX_SDA7
- U2 pad 24: Net-(U2-Pad24) -> /MUX_SCL7
- U2 pad 3: Net-(J2-Pad4) -> /ESP_SDA
- U2 pad 4: Net-(J2-Pad3) -> /ESP_SCL
- U2 pad 6: Net-(J3-Pad3) -> /V3V3
- U2 pad 7: Net-(J4-Pad4) -> GND
- U2 pad 8: Net-(J4-Pad3) -> GND
- U2 pad 9: GND -> Net-(U2-Pad9)
- U3 pad 1: Net-(U1-Pad28) -> GND
- U3 pad 2: Net-(U1-Pad29) -> /V3V3
- U3 pad 3: Net-(J1-Pad2) -> /ESP_SCL
- U3 pad 4: GND -> /ESP_SDA
- U4 pad 1: Net-(C1-Pad1) -> /V12V0IN
Routing:
- net Net-(C1-Pad1): track 448.9 -> 0.00 mm
- net /V12V0IN: track 0.00 -> 322.6 mm, vias 0 -> 6
- net /V3V3: track 0.00 -> 270.3 mm, vias 0 -> 6
- net Net-(J1-Pad2): track 267.5 -> 0.00 mm
- net Net-(U1-Pad29): track 167.1 -> 0.00 mm
- net GND: track 965.3 -> 801.2 mm, vias 0 -> 3
- net Net-(U1-Pad28): track 161.9 -> 0.00 mm
- net /ESP_SDA: track 0.00 -> 161.4 mm, vias 0 -> 2
- net /ESP_DEHUM_ON: track 0.00 -> 155.5 mm, vias 0 -> 2
- net /ESP_SCL: track 0.00 -> 154.9 mm, vias 0 -> 2
- net /ESP_FAN3_PWM: track 0.00 -> 114.5 mm, vias 0 -> 4
- net /ESP_CIRC_ON: track 184.1 -> 75.5 mm, vias 0 -> 2
- net Net-(Q6-Pad2): track 107.5 -> 0.00 mm
- net Net-(Q13-Pad2): track 89.9 -> 0.00 mm
- net Net-(J2-Pad3): track 76.3 -> 0.00 mm
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