File: Skizzen/Schaltplan/Schaltplan.sch (KiCad schematic (older format))
At the start: 0 parts

Commit message: Woche 2 29.09.2021 - 05.09.2021
-Code fertig
Parts:
- added U?: BME280 Inside, Package_LGA:Bosch_LGA-8_2.5x2.5mm_P0.65mm_ClockwisePinNumbering, symbol Sensor:BME280
- added U?: TCA9548A, Package_DFN_QFN:Texas_RGE0024C_EP2.1x2.1mm, symbol Interface_Expansion:TCA9548ARGER
- added U?: BME280 Outside, Package_LGA:Bosch_LGA-8_2.5x2.5mm_P0.65mm_ClockwisePinNumbering, symbol Sensor:BME280
- added U?: NodeMCU 0.9, RF_Module:ESP-12E, symbol RF_Module:ESP-12E
- added U?: RIT276-OLED-Display, symbol 0.92~Inch~OLED~Display:RIT276-OLED-Display
Connections:
- wire segments 0 -> 48
Changed lines of the file:
@@
 Comment4 ""
 $EndDescr
+$Comp
+L Interface_Expansion:TCA9548ARGER U?
+U 1 1 6133CE75
+P 5000 3550
+F 0 "U?" H 5000 4631 50  0000 C CNN
+F 1 "TCA9548A" H 5000 4540 50  0000 C CNN
+F 2 "Package_DFN_QFN:Texas_RGE0024C_EP2.1x2.1mm" H 5000 2550 50  0001 C CNN
+F 3 "http://www.ti.com/lit/ds/symlink/tca9548a.pdf" H 5050 3800 50  0001 C CNN
+	1    5000 3550
+	-1   0    0    1
+$EndComp
+$Comp
+L Sensor:BME280 U?
+U 1 1 6133FB63
+P 1150 3350
+F 0 "U?" V 675 3350 50  0000 C CNN
+F 1 "BME280 Outside" V 584 3350 50  0000 C CNN
+F 2 "Package_LGA:Bosch_LGA-8_2.5x2.5mm_P0.65mm_ClockwisePinNumbering" H 2650 2900 50  0001 C CNN
+F 3 "https://ae-bst.resource.bosch.com/media/_tech/media/datasheets/BST-BME280-DS002.pdf" H 1150 3150 50  0001 C CNN
+	1    1150 3350
+	1    0    0    -1
+$EndComp
+$Comp
+L RF_Module:ESP-12E U?
+U 1 1 61370196
+P 5000 5800
+F 0 "U?" H 5000 6781 50  0000 C CNN
+F 1 "NodeMCU 0.9" H 5000 6690 50  0000 C CNN
+F 2 "RF_Module:ESP-12E" H 5000 5800 50  0001 C CNN
+F 3 "http://wiki.ai-thinker.com/_media/esp8266/esp8266_series_modules_user_manual_v1.1.pdf" H 4650 5900 50  0001 C CNN
+	1    5000 5800
+	1    0    0    -1
+$EndComp
+$Comp
+L 0.92~Inch~OLED~Display:RIT276-OLED-Display U?
+U 1 1 6137AB6D
+P 6700 4100
+F 0 "U?" H 6978 3788 50  0000 L CNN
+F 1 "RIT276-OLED-Display" H 6978 3697 50  0000 L CNN
+F 2 "" H 6700 4100 50  0001 C CNN
+F 3 "" H 6700 4100 50  0001 C CNN
+	1    6700 4100
+	0    1    1    0
+$EndComp
+Wire Wire Line
+	5000 4450 5000 4750
+Wire Wire Line
+	5000 6500 4200 6500
+Wire Wire Line
+	1250 6500 1250 3950
+Wire Wire Line
+	1250 2750 3900 2750
+Wire Wire Line
+	3900 2750 3900 4750
+Wire Wire Line
+	3900 4750 5000 4750
+Connection ~ 5000 4750
+Wire Wire Line
+	5000 4750 5000 5000
+Wire Wire Line
+	6550 3550 6550 3700
+Wire Wire Line
+	6550 3700 5750 3700
+Wire Wire Line
+	5750 4750 5000 4750
+Wire Wire Line
+	6050 4150 5750 4150
+Wire Wire Line
+	5750 3700 5750 4150
+Connection ~ 5750 4150
+Wire Wire Line
+	5750 4150 5750 4750
+Wire Wire Line
+	5000 2550 4200 2550
+Connection ~ 4200 6500
+Wire Wire Line
+	4200 6500 1250 6500
+$Comp
+L Sensor:BME280 U?
+U 1 1 61336A88
+P 6650 2950
+F 0 "U?" V 6083 2950 50  0000 C CNN
+F 1 "BME280 Inside" V 6174 2950 50  0000 C CNN
+F 2 "Package_LGA:Bosch_LGA-8_2.5x2.5mm_P0.65mm_ClockwisePinNumbering" H 8150 2500 50  0001 C CNN
+F 3 "https://ae-bst.resource.bosch.com/media/_tech/media/datasheets/BST-BME280-DS002.pdf" H 6650 2750 50  0001 C CNN
+	1    6650 2950
+	-1   0    0    1
+$EndComp
+Wire Wire Line
+	6550 2350 5000 2350
+Wire Wire Line
+	5000 2350 5000 2550
+Connection ~ 5000 2550
+Wire Wire Line
+	6050 4250 6050 6500
+Wire Wire Line
+	6050 6500 5000 6500
+Connection ~ 5000 6500
+Wire Wire Line
+	4600 3850 2500 3850
+Wire Wire Line
+	2500 3850 2500 3250
+Wire Wire Line
+	2500 3250 1750 3250
+Wire Wire Line
+	1750 3450 2600 3450
+Wire Wire Line
+	2600 3450 2600 3750
+Wire Wire Line
+	2600 3750 4600 3750
+Wire Wire Line
+	4600 4250 4300 4250
+Wire Wire Line
+	4300 4250 4300 4650
+Wire Wire Line
+	4300 4650 5650 4650
+Wire Wire Line
+	5650 4050 6050 4050
+Wire Wire Line
+	6050 3950 5550 3950
+Wire Wire Line
+	5550 3950 5550 4900
+Wire Wire Line
+	4200 2550 4200 6500
+Wire Wire Line
+	4350 4900 4350 4150
+Wire Wire Line
+	4350 4150 4600 4150
+Wire Wire Line
+	4350 4900 5550 4900
+Wire Wire Line
+	4600 3950 4400 3950
+Wire Wire Line
+	4400 3950 4400 2450
+Wire Wire Line
+	4400 2450 5650 2450
+Wire Wire Line
+	5650 2450 5650 2850
+Wire Wire Line
+	5650 2850 6050 2850
+Wire Wire Line
+	6050 3050 5650 3050
+Wire Wire Line
+	5650 5000 5000 5000
+Wire Wire Line
+	4400 5000 4400 4050
+Wire Wire Line
+	4400 4050 4600 4050
+Wire Wire Line
+	5650 3050 5650 4050
+Connection ~ 5650 4050
+Wire Wire Line
+	5650 4050 5650 4650
+Connection ~ 5650 4650
+Wire Wire Line
+	5650 4650 5650 5000
+Connection ~ 5000 5000
+Wire Wire Line
+	5000 5000 4400 5000
 $EndSCHEMATC

Commit message: Woche 4 13.09.2021-20.09.2021
Parts:
- added C?: 100NF, symbol Device:C
- added M? (x2): Fan_4pin, symbol Motor:Fan_4pin
- added Q?: IRF9540N, Package_TO_SOT_THT:TO-220-3_Vertical, symbol Transistor_FET:IRF9540N
- added Q? (x3): 2N7000, Package_TO_SOT_THT:TO-92_Inline, symbol Transistor_FET:2N7000
- added R?: 3K9, symbol Device:R
- added R?: 1K1, symbol Device:R
Connections:
- net labels added: +12V, GND
- wire segments 48 -> 97

Commit message: Woche 5 19.09.2021 - 26.09.2021
Parts:
- added R?: 4K7, symbol Device:R
- added SW?: SW_Push, symbol Switch:SW_Push
Connections:
- wire segments 97 -> 105
Changed lines of the file:
@@
 Connection ~ 5000 4750
 Wire Wire Line
-	5000 4750 5000 5000
+	5000 4750 5000 4850
 Wire Wire Line
 	6550 3550 6550 3700
@@
 Wire Wire Line
 	5800 5700 5600 5700
-Wire Wire Line
-	5600 5900 7350 5900
-Wire Wire Line
-	7350 5900 7350 2250
 Connection ~ 7350 2250
 Wire Wire Line
@@
 $EndComp
 Wire Wire Line
-	10000 6500 6050 6500
+	10000 6500 6550 6500
 Connection ~ 6050 6500
 Wire Wire Line
@@
 Wire Wire Line
 	10300 1150 10100 1150
+Wire Wire Line
+	7350 2250 7350 5200
+Wire Wire Line
+	5600 5200 7350 5200
+$Comp
+L Switch:SW_Push SW?
+U 1 1 614D18A9
+P 7400 6000
+F 0 "SW?" H 7400 6285 50  0000 C CNN
+F 1 "SW_Push" H 7400 6194 50  0000 C CNN
+F 2 "" H 7400 6200 50  0001 C CNN
+F 3 "~" H 7400 6200 50  0001 C CNN
+	1    7400 6000
+	1    0    0    -1
+$EndComp
+Wire Wire Line
+	5600 6000 6550 6000
+Wire Wire Line
+	5000 4850 7600 4850
+Wire Wire Line
+	7600 4850 7600 6000
+Connection ~ 5000 4850
+Wire Wire Line
+	5000 4850 5000 5000
+$Comp
+L Device:R R?
+U 1 1 614DA686
+P 6550 6200
+F 0 "R?" H 6620 6246 50  0000 L CNN
+F 1 "4K7" H 6620 6155 50  0000 L CNN
+F 2 "" V 6480 6200 50  0001 C CNN
+F 3 "~" H 6550 6200 50  0001 C CNN
+	1    6550 6200
+	1    0    0    -1
+$EndComp
+Wire Wire Line
+	6550 6050 6550 6000
+Connection ~ 6550 6000
+Wire Wire Line
+	6550 6000 7200 6000
+Wire Wire Line
+	6550 6350 6550 6500
+Connection ~ 6550 6500
+Wire Wire Line
+	6550 6500 6050 6500
 $EndSCHEMATC

Commit message: Woche 7 01.10.2021 - 03.10.2021
Parts:
- removed C?: 100NF, symbol Device:C
- removed M? (x2): Fan_4pin, symbol Motor:Fan_4pin
- removed Q?: IRF9540N, Package_TO_SOT_THT:TO-220-3_Vertical, symbol Transistor_FET:IRF9540N
- removed Q? (x3): 2N7000, Package_TO_SOT_THT:TO-92_Inline, symbol Transistor_FET:2N7000
- removed R?: 3K9, symbol Device:R
- removed R?: 1K1, symbol Device:R
- removed R?: 4K7, symbol Device:R
- removed U?: BME280 Inside, Package_LGA:Bosch_LGA-8_2.5x2.5mm_P0.65mm_ClockwisePinNumbering, symbol Sensor:BME280
- removed U?: BME280 Outside, Package_LGA:Bosch_LGA-8_2.5x2.5mm_P0.65mm_ClockwisePinNumbering, symbol Sensor:BME280
- removed U?: NodeMCU 0.9, RF_Module:ESP-12E, symbol RF_Module:ESP-12E
- removed U?: RIT276-OLED-Display, symbol 0.92~Inch~OLED~Display:RIT276-OLED-Display
- added C1, C2, C3: 100NF, symbol Device:C
- added C4: 100nF, symbol Device:C
- added C5: 3.3uF, symbol Device:CP
- added J1, J2, J3, J4, J5, J6: I2C Sensor, symbol Connector_Generic:Conn_01x04
- added J10, J9: max. 250VAC/5A, TerminalBlock_RND:TerminalBlock_RND_205-00001_1x02_P5.00mm_Horizontal, symbol Connector:Screw_Terminal_01x02
- added J7: 12V DC, 2A, symbol Connector:Barrel_Jack_Switch
- added J8: max. 30VDC/2A, TerminalBlock_RND:TerminalBlock_RND_205-00002_1x03_P5.00mm_Horizontal, symbol Connector:Screw_Terminal_01x03
- added K1, K2: G5LE-1, Relay_THT:Relay_SPDT_Omron-G5LE-1, symbol Relay:G5LE-1
- added K3: G6S-2, symbol Relay:G6S-2
- added M1: FAN0, Connector_PinSocket_2.54mm:PinSocket_1x04_P2.54mm_Vertical, symbol Motor:Fan_4pin
- added M2: FAN1, Connector_PinSocket_2.54mm:PinSocket_1x04_P2.54mm_Vertical, symbol Motor:Fan_4pin
- added M3: FAN2, Connector_PinSocket_2.54mm:PinSocket_1x04_P2.54mm_Vertical, symbol Motor:Fan_4pin
- added Q1, Q13, Q14, Q15, Q2, Q3, Q4, Q5, Q6, Q7, Q8, Q9: 2N7000, Package_TO_SOT_THT:TO-92_Inline, symbol Transistor_FET:2N7000
- added Q10, Q11, Q12: IRF9540N, Package_TO_SOT_THT:TO-220-3_Vertical, symbol Transistor_FET:IRF9540N
- added R1: 10k, symbol Device:R
- added R10, R6, R8: 1K1, symbol Device:R
- added R11: 240R, symbol Device:R
- added R2, R3, R4: 4K7, symbol Device:R
- added R5, R7, R9: 3K9, symbol Device:R
- added U1: NodeMCU_1.0_(ESP-12E), ESP8266:ESP12F-Devkit-V3, symbol Schaltplan-rescue:NodeMCU_1.0_(ESP-12E)-ESP8266
- added U3: RIT276-OLED-Display, Connector_PinHeader_2.54mm:PinHeader_1x04_P2.54mm_Vertical, symbol Schaltplan-rescue:RIT276-OLED-Display-0.92_Inch_OLED_Display
- added U4: LM7805_TO220, Package_TO_SOT_THT:TO-220-3_Vertical, symbol Regulator_Linear:LM7805_TO220
- SW1: renamed from SW?; value SW_Push -> CFG_MODE; footprint (none) -> Connector_PinHeader_2.54mm:PinHeader_1x02_P2.54mm_Vertical
- gave numbers to parts that had none: 1
Connections:
- net labels removed: +12V
- wire segments 105 -> 268
- no-connect marks 0 -> 20
Other:
- note added: "Arduino GPIO\nD0\nD1\nD2\nD3\nD4\nD5\nD6\nD7\nD8\nD9/RX\nD10/TX\nD11/SD2\nD12/SD3"
- note added: "Board Usage\n-\nI2C_SCL\nI2C_SDA\nCirculation Pump On\nExt. Dehumidifier\nFAN1 PWM\nFAN2 PWM\nFAN3 PWM\nCFG_MODE\n-\n-\n-\n-"
- note added: "Circulation Pump\nfor heat exchanger."
- note added: "D4=External Dehumidifier ON"
- note added: "Ext. Dehumidifier\nTank Full Signal."
- note added: "Ext. Power Outlet\nfor Dehumidifier."
- note added: "GND\nVCC\nSCL\nSDA"
- note added: "GPIO Mapping:"
- note added: "NodeMCU Pin\nGPIO16\nGPIO5\nGPIO4\nGPIO0\nGPIO2\nGPIO14\nGPIO12\nGPIO13\nGPIO15\nGPIO3\nGPIO1\nGPIO9\nGPIO10"
- moved on the sheet: SW1, U2

Commit message: Woche 8 10.10.2021 - 17.10.2021
Parts:
- C1, C2, C3, C4: footprint (none) -> Capacitor_THT:C_Disc_D4.3mm_W1.9mm_P5.00mm
- C5: footprint (none) -> Capacitor_THT:C_Disc_D3.0mm_W1.6mm_P2.50mm
- J1, J2, J3, J4, J5, J6: footprint (none) -> Sensor:Aosong_DHT11_5.5x12.0_P2.54mm
- J7: footprint (none) -> Jumper:SolderJumper-3_P1.3mm_Bridged12_Pad1.0x1.5mm
- K3: footprint (none) -> Relay_THT:Relay_DPDT_Omron_G6S-2
- R1, R10, R2, R3, R4, R5, R6, R7, R8, R9: footprint (none) -> Resistor_THT:R_Axial_DIN0204_L3.6mm_D1.6mm_P7.62mm_Horizontal
- R11: footprint (none) -> Resistor_THT:R_Axial_DIN0207_L6.3mm_D2.5mm_P7.62mm_Horizontal
- U2: footprint Package_DFN_QFN:Texas_RGE0024C_EP2.1x2.1mm -> KL:TCA9548A
Changed lines of the file:
@@
 F 0 "U2" H 5700 6631 50  0000 C CNN
 F 1 "TCA9548A" H 5700 6540 50  0000 C CNN
-F 2 "Package_DFN_QFN:Texas_RGE0024C_EP2.1x2.1mm" H 5700 4550 50  0001 C CNN
+F 2 "KL:TCA9548A" H 5700 4550 50  0001 C CNN
 F 3 "http://www.ti.com/lit/ds/symlink/tca9548a.pdf" H 5750 5800 50  0001 C CNN
 	1    5700 5550
@@
 F 0 "K3" H 13630 5196 50  0000 L CNN
 F 1 "G6S-2" H 13630 5105 50  0000 L CNN
-F 2 "" H 13000 5150 50  0001 L CNN
+F 2 "Relay_THT:Relay_DPDT_Omron_G6S-2" H 13000 5150 50  0001 L CNN
 F 3 "http://omronfs.omron.com/en_US/ecb/products/pdf/en-g6s.pdf" H 13000 5150 50  0001 C CNN
 	1    13000 5150
@@
 F 0 "J7" H 14820 1592 50  0000 R CNN
 F 1 "12V DC, 2A" H 14820 1501 50  0000 R CNN
-F 2 "" H 15100 1510 50  0001 C CNN
+F 2 "Jumper:SolderJumper-3_P1.3mm_Bridged12_Pad1.0x1.5mm" H 15100 1510 50  0001 C CNN
 F 3 "~" H 15100 1510 50  0001 C CNN
 	1    15050 1550
@@
 F 0 "C5" H 14068 1646 50  0000 L CNN
 F 1 "3.3uF" H 14068 1555 50  0000 L CNN
-F 2 "" H 13988 1450 50  0001 C CNN
+F 2 "Capacitor_THT:C_Disc_D3.0mm_W1.6mm_P2.50mm" H 13988 1450 50  0001 C CNN
 F 3 "~" H 13950 1600 50  0001 C CNN
 	1    13950 1600
@@
 F 0 "C4" H 13015 1646 50  0000 L CNN
 F 1 "100nF" H 13015 1555 50  0000 L CNN
-F 2 "" H 12938 1450 50  0001 C CNN
+F 2 "Capacitor_THT:C_Disc_D4.3mm_W1.9mm_P5.00mm" H 12938 1450 50  0001 C CNN
 F 3 "~" H 12900 1600 50  0001 C CNN
 	1    12900 1600
@@
 F 0 "R11" H 12670 5646 50  0000 L CNN
 F 1 "240R" H 12670 5555 50  0000 L CNN
-F 2 "" V 12530 5600 50  0001 C CNN
+F 2 "Resistor_THT:R_Axial_DIN0207_L6.3mm_D2.5mm_P7.62mm_Horizontal" V 12530 5600 50  0001 C CNN
 F 3 "~" H 12600 5600 50  0001 C CNN
 	1    12600 5600
@@
 F 0 "R5" H 9320 1546 50  0000 L CNN
 F 1 "3K9" H 9320 1455 50  0000 L CNN
-F 2 "" V 9180 1500 50  0001 C CNN
+F 2 "Resistor_THT:R_Axial_DIN0204_L3.6mm_D1.6mm_P7.62mm_Horizontal" V 9180 1500 50  0001 C CNN
 F 3 "~" H 9250 1500 50  0001 C CNN
 	1    9250 1500
@@
 F 0 "C1" H 9715 1546 50  0000 L CNN
 F 1 "100NF" H 9715 1455 50  0000 L CNN
-F 2 "" H 9638 1350 50  0001 C CNN
+F 2 "Capacitor_THT:C_Disc_D4.3mm_W1.9mm_P5.00mm" H 9638 1350 50  0001 C CNN
 F 3 "~" H 9600 1500 50  0001 C CNN
 	1    9600 1500
@@
 F 0 "R6" H 9320 1946 50  0000 L CNN
 F 1 "1K1" H 9320 1855 50  0000 L CNN
-F 2 "" V 9180 1900 50  0001 C CNN
+F 2 "Resistor_THT:R_Axial_DIN0204_L3.6mm_D1.6mm_P7.62mm_Horizontal" V 9180 1900 50  0001 C CNN
 F 3 "~" H 9250 1900 50  0001 C CNN
 	1    9250 1900
@@
 F 0 "R2" H 8470 1346 50  0000 L CNN
 F 1 "4K7" H 8470 1255 50  0000 L CNN
-F 2 "" V 8330 1300 50  0001 C CNN
+F 2 "Resistor_THT:R_Axial_DIN0204_L3.6mm_D1.6mm_P7.62mm_Horizontal" V 8330 1300 50  0001 C CNN
 F 3 "~" H 8400 1300 50  0001 C CNN
 	1    8400 1300
@@
 F 0 "R7" H 9320 3246 50  0000 L CNN
 F 1 "3K9" H 9320 3155 50  0000 L CNN
-F 2 "" V 9180 3200 50  0001 C CNN
+F 2 "Resistor_THT:R_Axial_DIN0204_L3.6mm_D1.6mm_P7.62mm_Horizontal" V 9180 3200 50  0001 C CNN
 F 3 "~" H 9250 3200 50  0001 C CNN
 	1    9250 3200
@@
 F 0 "C2" H 9715 3246 50  0000 L CNN
 F 1 "100NF" H 9715 3155 50  0000 L CNN
-F 2 "" H 9638 3050 50  0001 C CNN
+F 2 "Capacitor_THT:C_Disc_D4.3mm_W1.9mm_P5.00mm" H 9638 3050 50  0001 C CNN
 F 3 "~" H 9600 3200 50  0001 C CNN
 	1    9600 3200
@@
 F 0 "R8" H 9320 3646 50  0000 L CNN
 F 1 "1K1" H 9320 3555 50  0000 L CNN
-F 2 "" V 9180 3600 50  0001 C CNN
+F 2 "Resistor_THT:R_Axial_DIN0204_L3.6mm_D1.6mm_P7.62mm_Horizontal" V 9180 3600 50  0001 C CNN
 F 3 "~" H 9250 3600 50  0001 C CNN
 	1    9250 3600
@@
 F 0 "R3" H 8470 3046 50  0000 L CNN
 F 1 "4K7" H 8470 2955 50  0000 L CNN
-F 2 "" V 8330 3000 50  0001 C CNN
+F 2 "Resistor_THT:R_Axial_DIN0204_L3.6mm_D1.6mm_P7.62mm_Horizontal" V 8330 3000 50  0001 C CNN
 F 3 "~" H 8400 3000 50  0001 C CNN
 	1    8400 3000
@@
 F 0 "R9" H 9320 4946 50  0000 L CNN
 F 1 "3K9" H 9320 4855 50  0000 L CNN
-F 2 "" V 9180 4900 50  0001 C CNN
+F 2 "Resistor_THT:R_Axial_DIN0204_L3.6mm_D1.6mm_P7.62mm_Horizontal" V 9180 4900 50  0001 C CNN
 F 3 "~" H 9250 4900 50  0001 C CNN
 	1    9250 4900
@@
 F 0 "C3" H 9715 4946 50  0000 L CNN
 F 1 "100NF" H 9715 4855 50  0000 L CNN
-F 2 "" H 9638 4750 50  0001 C CNN
+F 2 "Capacitor_THT:C_Disc_D4.3mm_W1.9mm_P5.00mm" H 9638 4750 50  0001 C CNN
 F 3 "~" H 9600 4900 50  0001 C CNN
 	1    9600 4900
@@
 F 0 "R10" H 9320 5346 50  0000 L CNN
 F 1 "1K1" H 9320 5255 50  0000 L CNN
-F 2 "" V 9180 5300 50  0001 C CNN
+F 2 "Resistor_THT:R_Axial_DIN0204_L3.6mm_D1.6mm_P7.62mm_Horizontal" V 9180 5300 50  0001 C CNN
 F 3 "~" H 9250 5300 50  0001 C CNN
 	1    9250 5300
@@
 F 0 "R4" H 8470 4746 50  0000 L CNN
 F 1 "4K7" H 8470 4655 50  0000 L CNN
-F 2 "" V 8330 4700 50  0001 C CNN
+F 2 "Resistor_THT:R_Axial_DIN0204_L3.6mm_D1.6mm_P7.62mm_Horizontal" V 8330 4700 50  0001 C CNN
 F 3 "~" H 8400 4700 50  0001 C CNN
 	1    8400 4700
@@
 F 0 "J1" H 1168 5267 50  0000 C CNN
 F 1 "I2C Sensor" H 1168 5176 50  0000 C CNN
-F 2 "" H 1250 4950 50  0001 C CNN
+F 2 "Sensor:Aosong_DHT11_5.5x12.0_P2.54mm" H 1250 4950 50  0001 C CNN
 F 3 "~" H 1250 4950 50  0001 C CNN
 	1    1250 4950
@@
 F 0 "J2" H 1168 5917 50  0000 C CNN
 F 1 "I2C Sensor" H 1168 5826 50  0000 C CNN
-F 2 "" H 1250 5600 50  0001 C CNN
+F 2 "Sensor:Aosong_DHT11_5.5x12.0_P2.54mm" H 1250 5600 50  0001 C CNN
 F 3 "~" H 1250 5600 50  0001 C CNN
 	1    1250 5600
@@
 F 0 "J3" H 1168 6567 50  0000 C CNN
 F 1 "I2C Sensor" H 1168 6476 50  0000 C CNN
-F 2 "" H 1250 6250 50  0001 C CNN
+F 2 "Sensor:Aosong_DHT11_5.5x12.0_P2.54mm" H 1250 6250 50  0001 C CNN
 F 3 "~" H 1250 6250 50  0001 C CNN
 	1    1250 6250
@@
 F 0 "J4" H 1168 7217 50  0000 C CNN
 F 1 "I2C Sensor" H 1168 7126 50  0000 C CNN
-F 2 "" H 1250 6900 50  0001 C CNN
+F 2 "Sensor:Aosong_DHT11_5.5x12.0_P2.54mm" H 1250 6900 50  0001 C CNN
 F 3 "~" H 1250 6900 50  0001 C CNN
 	1    1250 6900
@@
 F 0 "J5" H 1168 7867 50  0000 C CNN
 F 1 "I2C Sensor" H 1168 7776 50  0000 C CNN
-F 2 "" H 1250 7550 50  0001 C CNN
+F 2 "Sensor:Aosong_DHT11_5.5x12.0_P2.54mm" H 1250 7550 50  0001 C CNN
 F 3 "~" H 1250 7550 50  0001 C CNN
 	1    1250 7550
@@
 F 0 "J6" H 1168 8517 50  0000 C CNN
 F 1 "I2C Sensor" H 1168 8426 50  0000 C CNN
-F 2 "" H 1250 8200 50  0001 C CNN
+F 2 "Sensor:Aosong_DHT11_5.5x12.0_P2.54mm" H 1250 8200 50  0001 C CNN
 F 3 "~" H 1250 8200 50  0001 C CNN
 	1    1250 8200
@@
 F 0 "R1" H 6920 3546 50  0000 L CNN
 F 1 "10k" H 6920 3455 50  0000 L CNN
-F 2 "" V 6780 3500 50  0001 C CNN
+F 2 "Resistor_THT:R_Axial_DIN0204_L3.6mm_D1.6mm_P7.62mm_Horizontal" V 6780 3500 50  0001 C CNN
 F 3 "~" H 6850 3500 50  0001 C CNN
 	1    6850 3500

Commit message: Woche 9 17.10.2021 - 24.10.2021
Parts:
- J7: footprint Jumper:SolderJumper-3_P1.3mm_Bridged12_Pad1.0x1.5mm -> KL:Buchse
Connections:
- net at C1.1, C3.1, C5.1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: now also C2.1, Q11.2 (D), R7.1
Changed lines of the file:
@@
 F 0 "J7" H 14820 1592 50  0000 R CNN
 F 1 "12V DC, 2A" H 14820 1501 50  0000 R CNN
-F 2 "Jumper:SolderJumper-3_P1.3mm_Bridged12_Pad1.0x1.5mm" H 15100 1510 50  0001 C CNN
+F 2 "KL:Buchse" H 15100 1510 50  0001 C CNN
 F 3 "~" H 15100 1510 50  0001 C CNN
 	1    15050 1550
@@
 Wire Wire Line
 	12650 8250 12650 8450
-Wire Wire Line
-	14150 650  14150 1450
-Wire Wire Line
-	13950 1450 14150 1450
-Wire Wire Line
-	14150 1450 14350 1450
-Connection ~ 14150 1450
 Wire Wire Line
 	11850 5950 12300 5950
@@
 $EndComp
 Wire Wire Line
-	9950 650  10500 650
-Wire Wire Line
 	15150 2050 13850 2050
 Wire Wire Line
@@
 Wire Wire Line
 	8400 4450 9300 4450
-Wire Wire Line
-	9950 2950 10500 2950
-Connection ~ 9950 2950
-Connection ~ 10500 650
-Wire Wire Line
-	10500 650  14150 650
 $Comp
 L Transistor_FET:IRF9540N Q12
@@
 Connection ~ 9950 4650
 Wire Wire Line
-	10500 650  10500 4650
-Wire Wire Line
 	11400 4550 11400 3850
 Wire Wire Line
@@
 Wire Wire Line
 	3000 2950 3000 1000
-Wire Wire Line
-	3000 1000 12900 1000
-Wire Wire Line
-	12900 1000 12900 1450
-Connection ~ 12900 1450
 Wire Wire Line
 	6200 2950 6200 4650
@@
 Wire Notes Line
 	6150 9750 6150 10950
+Connection ~ 12900 1450
+Connection ~ 14150 1450
+Wire Wire Line
+	14150 1450 14350 1450
+Wire Wire Line
+	13950 1450 14150 1450
+Wire Wire Line
+	12900 1000 12900 1450
+Wire Wire Line
+	3000 1000 12900 1000
+Wire Wire Line
+	10500 650  10500 2950
+Wire Wire Line
+	10500 650  14150 650
+Connection ~ 10500 650
+Wire Wire Line
+	9950 650  10500 650
+Wire Wire Line
+	14150 650  14150 1450
+Wire Wire Line
+	9950 2950 10500 2950
+Connection ~ 9950 2950
+Connection ~ 10500 2950
+Wire Wire Line
+	10500 2950 10500 4650
 $EndSCHEMATC
