File: Skizzen/Schaltplan/Schaltplan.sch (KiCad schematic (older format))
At the start: 52 parts, among them J1 I2C Sensor, J10 max. 250VAC/5A, J2 I2C Sensor, J3 I2C Sensor, J4 I2C Sensor, J5 I2C Sensor, J6 I2C Sensor, J7 12V DC, 2A, J8 max. 30VDC/2A, J9 max. 250VAC/5A, K1 G5LE-1, K2 G5LE-1, K3 G6S-2, M1 FAN0, M2 FAN1, M3 FAN2, Q1 2N7000, Q10 IRF9540N, Q11 IRF9540N, Q12 IRF9540N, Q13 2N7000, Q14 2N7000, Q15 2N7000, Q2 2N7000, Q3 2N7000, Q4 2N7000, Q5 2N7000, Q6 2N7000, Q7 2N7000, Q8 2N7000, Q9 2N7000, SW1 CFG_MODE, U1 NodeMCU_1.0_(ESP-12E), U2 TCA9548A, U3 RIT276-OLED-Display, U4 LM7805_TO220

Commit message: Woche 20 02.01.2022 - 08.01.2022
Parts:
- removed J1, J2, J3, J4, J5, J6: I2C Sensor, Sensor:Aosong_DHT11_5.5x12.0_P2.54mm, symbol Connector_Generic:Conn_01x04
- removed U2: TCA9548A, KL:TCA9548A, symbol Interface_Expansion:TCA9548ARGER
- added H1, H2, H3, H4: MountingHole, MountingHole:MountingHole_3.2mm_M3, symbol Mechanical:MountingHole
- added J1: Conn_02x24_Counter_Clockwise, Terminals:FFKDSH-2,54_24, symbol Connector_Generic:Conn_02x24_Counter_Clockwise
- added U2: TCA9548A_Breakout, KL:TCA9548A_Breakout, symbol KL2021:TCA9548A_Breakout
- added U5: YAAJ_DCDC_StepDown_LM2596, LM2596Module:YAAJ_DCDC_StepDown_LM2596, symbol yaaj_dcdc_stepdown_lm2596:YAAJ_DCDC_StepDown_LM2596
- C5: footprint Capacitor_THT:C_Disc_D3.0mm_W1.6mm_P2.50mm -> Capacitor_THT:CP_Radial_Tantal_D4.5mm_P5.00mm
- J7: footprint KL:Buchse -> Connector_PinHeader_2.54mm:PinHeader_1x03_P2.54mm_Vertical
- M1: value FAN0 -> FAN1
- M2: value FAN1 -> FAN2
- M3: value FAN2 -> FAN3
- R1, R2, R3, R4, R5, R7, R9: footprint Resistor_THT:R_Axial_DIN0204_L3.6mm_D1.6mm_P7.62mm_Horizontal -> Resistor_THT:R_Axial_DIN0204_L3.6mm_D1.6mm_P2.54mm_Vertical
- R11: footprint Resistor_THT:R_Axial_DIN0207_L6.3mm_D2.5mm_P7.62mm_Horizontal -> Resistor_THT:R_Axial_DIN0204_L3.6mm_D1.6mm_P2.54mm_Vertical
- U3: footprint Connector_PinHeader_2.54mm:PinHeader_1x04_P2.54mm_Vertical -> Oled-Display:SSD1306_128x64_0.96; symbol Schaltplan-rescue:RIT276-OLED-Display-0.92_Inch_OLED_Display -> 0.92_Inch_OLED_Display:RIT276-OLED-Display
Connections:
- net GND: now also U3.1 (GND), J1.1 (Pin_1), J1.13 (Pin_13), J1.17 (Pin_17), J1.21 (Pin_21), J1.5 (Pin_5), J1.9 (Pin_9), U2.2 (GND), U2.7 (A1), U2.8 (A2), U5.2 (GND), U5.3 (GND); no longer U3.4 (GND)
- net ESP_SCL: now reaches U1.29 (D1(GPIO5))
- net ESP_SCL: now also U3.3 (SCL), U2.4 (SCL); no longer U3.2 (SCL)
- net ESP_SDA: now reaches U1.28 (D2(GPIO4))
- net ESP_SDA: now also U3.4 (SDA), U2.3 (SDA); no longer U3.1 (SDA)
- net V3V3: now reaches R1.1, U1.11 (3.3V), U1.16 (3.3V), U1.25 (3.3V)
- net V3V3: now also U3.2 (VCC), J1.10 (Pin_10), J1.14 (Pin_14), J1.18 (Pin_18), J1.2 (Pin_2), J1.22 (Pin_22), J1.6 (Pin_6), U2.1 (VCC), U2.6 (A0); no longer U3.3 (VCC)
- net ESP_FORCE_CFG_MODE: now reaches R1.2, SW1.1
- net ESP_FORCE_CFG_MODE: now also U1.21 (D7(GPIO13)); no longer U1.20 (D8(GPIO15))
- net V12V0IN: now reaches C1.1, C2.1, C3.1, C5.1, J7.1, K2.5, K3.1, R5.1, R7.1, R9.1, U4.1 (VI)
- net V12V0IN: now also K1.2, Q10.3 (S), Q11.3 (S), Q12.3 (S), R2.1, R3.1, R4.1, U5.1 (Vin); no longer K1.5, Q10.2 (D), Q11.2 (D), Q12.2 (D)
- net at K3.10: now also J8.3 (Pin_3); no longer J8.1 (Pin_1)
- net TANK_FULL_CLOSE: now reaches K3.8
- net TANK_FULL_CLOSE: now also J8.1 (Pin_1); no longer J8.2 (Pin_2)
- net TANK_FULL_COMMON: now reaches K3.9
- net TANK_FULL_COMMON: now also J8.2 (Pin_2); no longer J8.3 (Pin_3)
- net at Q14.3 (D): now also K1.5; no longer K1.2
- net V5V0: now reaches C4.1, U1.15 (VIN), U4.3 (VO)
- net V5V0: now also U5.4 (Vout)
- net ESP_DEHUM_ON: now reaches Q13.2 (G), Q14.2 (G)
- net ESP_DEHUM_ON: now also U1.4 (SD3(GPIO10)); no longer U1.26 (D4(GPIO2))
- net ESP_CIRC_ON: now reaches Q15.2 (G), U1.27 (D3(GPIO0))
- net FAN1_V12V0: now reaches M1.2 (+)
- net FAN1_V12V0: now also Q10.2 (D); no longer Q10.3 (S)
- net FAN1_PWM: now reaches M1.4 (PWM), Q1.3 (D)
- net FAN1_PWM: no longer R2.1
- net FAN2_V12V0: now reaches M2.2 (+)
- net FAN2_V12V0: now also Q11.2 (D); no longer Q11.3 (S)
- net FAN2_PWM: now reaches M2.4 (PWM), Q3.3 (D)
- net FAN2_PWM: no longer R3.1
- net at M3.2 (+): now also Q12.2 (D); no longer Q12.3 (S)
- net FAN3_PWM: now reaches M3.4 (PWM), Q5.3 (D)
- net FAN3_PWM: no longer R4.1
- net ESP_FAN1_PWM: now reaches Q2.2 (G), Q7.2 (G), U1.23 (D5(GPIO14))
- net FAN1_PWM#: now reaches Q1.2 (G), Q2.3 (D), R2.2
- net ESP_FAN2_PWM: now reaches Q4.2 (G), Q8.2 (G), U1.22 (D6(GPIO12))
- net FAN2_PWM#: now reaches Q3.2 (G), Q4.3 (D), R3.2
- net ESP_FAN3_PWM: now reaches Q6.2 (G), Q9.2 (G)
- net ESP_FAN3_PWM: now also U1.20 (D8(GPIO15)); no longer U1.21 (D7(GPIO13))
- net FAN3_PWM#: now reaches Q5.2 (G), Q6.3 (D), R4.2
- new net MUX_SCL2: J1.45 (Pin_45), U2.14 (SC2)
- new net MUX_SCL3: J1.41 (Pin_41), U2.16 (SC3)
- new net MUX_SCL4: J1.37 (Pin_37), U2.18 (SC4)
- new net MUX_SCL5: J1.33 (Pin_33), U2.20 (SC5)
- new net MUX_SCL6: J1.29 (Pin_29), U2.22 (SC6)
- new net MUX_SCL7: J1.25 (Pin_25), U2.24 (SC7)
- new net MUX_SDA2: J1.46 (Pin_46), U2.13 (SD2)
- new net MUX_SDA3: J1.42 (Pin_42), U2.15 (SD3)
- new net MUX_SDA4: J1.38 (Pin_38), U2.17 (SD4)
- new net MUX_SDA5: J1.34 (Pin_34), U2.19 (SD5)
- new net MUX_SDA6: J1.30 (Pin_30), U2.21 (SD6)
- new net MUX_SDA7: J1.26 (Pin_26), U2.23 (SD7)
- no-connect marks 20 -> 51
Other:
- note added: "Board Usage\n-\nI2C_SCL\nI2C_SDA\nCirculation Pump On\n-\nFAN1 PWM\nFAN2 PWM\nCFG_MODE\nFAN3 PWM\n-\n-\n-\nExt. Dehumidifier"
- note added: "Device\nI2C Mux\nDisplay\nOut BME280\nIn BME280\nWall LM75\n\n\n\n\n\n\n\n\n"
- note added: "I2C Busses:"
- note added: "I2C-Address (7-Bit)\n0x71\n0x3C\n0x76\n0x76\n0x48\n\n\n\n\n\n\n\n\n"
- note added: "I2C-Bus\nESP I2C\nESP I2C\nMux Ch. 2\nMux Ch. 3\nMux Ch. 4\n\n\n\n\n\n\n\n\n"
- note added: "SD3/GPIO10=External Dehumidifier ON"
- note removed: "Board Usage\n-\nI2C_SCL\nI2C_SDA\nCirculation Pump On\nExt. Dehumidifier\nFAN1 PWM\nFAN2 PWM\nFAN3 PWM\nCFG_MODE\n-\n-\n-\n-"
- note removed: "D4=External Dehumidifier ON"
- moved on the sheet: Q14
